File: CAN_board/CAN_board.sch (KiCad schematic (older format))
At the start: 7 parts, among them J1 Conn_02x20_Odd_Even_Rasbpi, J2 Conn_02x20_Odd_Even_extra, J3 Converter, J4 MCP2515, J5 Battery, J6 Conn_01x02_Male, J7 OBD_connector

Commit message: Components placed, routing to be done
Parts:
- removed J2: Conn_02x20_Odd_Even_extra, Connector_PinHeader_2.54mm:PinHeader_2x20_P2.54mm_Vertical, symbol Connector_Generic:Conn_02x20_Odd_Even
- removed J3: Converter, Connector_PinHeader_2.54mm:PinHeader_1x04_P2.54mm_Vertical, symbol Connector:Conn_01x04_Male
- removed J7: OBD_connector, Connector_PinHeader_2.54mm:PinHeader_1x09_P2.54mm_Vertical, symbol Connector:Conn_01x09_Male
- added J2: Sensor input, Connector_PinHeader_2.54mm:PinHeader_1x04_P2.54mm_Vertical, symbol Connector:Conn_01x04_Male
- added J3: ADS1115, Connector_PinHeader_2.54mm:PinHeader_1x10_P2.54mm_Vertical, symbol Connector:Conn_01x10_Female
- added J7: Conn_01x02_Male, Connector_PinHeader_2.54mm:PinHeader_1x02_P2.54mm_Vertical, symbol Connector:Conn_01x02_Male
Connections:
- net labels added: A0, A1, A2, A3, ALRT, SCL, SDA
- net labels removed: 11, 12V, 3, 5, ISO9141-2-K-line, ISO9141-2L
Changed lines of the file:
@@
 EESchema Schematic File Version 4
-EELAYER 26 0
+LIBS:CAN_board-cache
+EELAYER 29 0
 EELAYER END
 $Descr A4 11693 8268
@@
 $EndDescr
 $Comp
-L Connector_Generic:Conn_02x20_Odd_Even J2
-U 1 1 5C177763
-P 2400 3150
-F 0 "J2" H 2450 4267 50  0000 C CNN
-F 1 "Conn_02x20_Odd_Even_extra" H 2550 4350 50  0000 C CNN
-F 2 "Connector_PinHeader_2.54mm:PinHeader_2x20_P2.54mm_Vertical" H 2400 3150 50  0001 C CNN
-F 3 "~" H 2400 3150 50  0001 C CNN
-	1    2400 3150
-	1    0    0    -1
-$EndComp
-Text Label 2200 2250 2    50   ~ 0
-3V3
-Text Label 2700 2250 0    50   ~ 0
-5V
-Text Label 2700 2450 0    50   ~ 0
-GND
-Text Label 2200 3150 2    50   ~ 0
-MOSI
-Text Label 2200 3250 2    50   ~ 0
-MISO
-Text Label 2200 3350 2    50   ~ 0
-SCLK
-$Comp
 L Connector:Conn_01x08_Female J4
 U 1 1 5C1778C2
@@
 Text Label 3850 2200 2    50   ~ 0
 5V
-Text Label 2700 3350 0    50   ~ 0
-CS
-Text Label 2700 3250 0    50   ~ 0
-INT
-$Comp
-L Connector:Conn_01x04_Male J3
-U 1 1 5C177A3F
-P 3450 3650
-F 0 "J3" H 3556 3928 50  0000 C CNN
-F 1 "Converter" H 3556 3837 50  0000 C CNN
-F 2 "Connector_PinHeader_2.54mm:PinHeader_1x04_P2.54mm_Vertical" H 3450 3650 50  0001 C CNN
-F 3 "~" H 3450 3650 50  0001 C CNN
-	1    3450 3650
-	1    0    0    -1
-$EndComp
-Text Label 3650 3550 0    50   ~ 0
-12V
-Text Label 3650 3650 0    50   ~ 0
-12V
-Text Label 3650 3750 0    50   ~ 0
-GND
-Text Label 3650 3850 0    50   ~ 0
-GND
 $Comp
 L Connector:Conn_01x04_Male J5
@@
 $EndComp
 Text Label 4600 3550 0    50   ~ 0
-12V
+5V
 Text Label 4600 3650 0    50   ~ 0
-12V
+3V3
 Text Label 4600 3750 0    50   ~ 0
 GND
 Text Label 4600 3850 0    50   ~ 0
 GND
-$Comp
-L Connector:Conn_01x09_Male J7
-U 1 1 5C177B72
-P 5300 3200
-F 0 "J7" H 5406 3778 50  0000 C CNN
-F 1 "OBD_connector" H 5406 3687 50  0000 C CNN
-F 2 "Connector_PinHeader_2.54mm:PinHeader_1x09_P2.54mm_Vertical" H 5300 3200 50  0001 C CNN
-F 3 "~" H 5300 3200 50  0001 C CNN
-	1    5300 3200
-	1    0    0    -1
-$EndComp
-Text Label 5500 3100 0    50   ~ 0
-CANL
-Text Label 5500 3200 0    50   ~ 0
-GND
-Text Label 5500 3300 0    50   ~ 0
-ISO9141-2L
-Text Label 5500 3400 0    50   ~ 0
-CANH
-Text Label 5500 3500 0    50   ~ 0
-12V
-Text Label 5500 3600 0    50   ~ 0
-ISO9141-2-K-line
 $Comp
 L Connector:Conn_01x02_Male J6
@@
 Text Label 5300 2250 0    50   ~ 0
 CANL
-Text Label 2200 2350 2    50   ~ 0
-3
-Text Label 2200 2450 2    50   ~ 0
-5
-Text Label 2200 2550 2    50   ~ 0
-7
-Text Label 2200 2750 2    50   ~ 0
-11
-Text Label 2200 2850 2    50   ~ 0
-13
-Text Label 2200 2950 2    50   ~ 0
-15
-Text Label 2200 3550 2    50   ~ 0
-27
-Text Label 2200 3650 2    50   ~ 0
-29
-Text Label 2200 3750 2    50   ~ 0
-31
-Text Label 2200 3850 2    50   ~ 0
-33
-Text Label 2200 3950 2    50   ~ 0
-35
-Text Label 2200 4050 2    50   ~ 0
-37
-Text Label 2700 2550 0    50   ~ 0
-8
-Text Label 2700 2650 0    50   ~ 0
-10
-Text Label 2700 2750 0    50   ~ 0
-12
-Text Label 2700 2950 0    50   ~ 0
-16
-Text Label 2700 3050 0    50   ~ 0
-18
-Text Label 2700 3450 0    50   ~ 0
-26
-Text Label 2700 3550 0    50   ~ 0
-28
-Text Label 2700 3750 0    50   ~ 0
-32
-Text Label 2700 3950 0    50   ~ 0
-36
-Text Label 2700 4050 0    50   ~ 0
-38
-Text Label 2700 4150 0    50   ~ 0
-40
-Text Label 2700 2350 0    50   ~ 0
-5V
-Text Label 2200 2650 2    50   ~ 0
-GND
-Text Label 2700 2850 0    50   ~ 0
-GND
-Text Label 2700 3150 0    50   ~ 0
-GND
-Text Label 2200 3050 2    50   ~ 0
-3V3
-Text Label 2200 3450 2    50   ~ 0
-GND
-Text Label 2700 3650 0    50   ~ 0
-GND
-Text Label 2700 3850 0    50   ~ 0
-GND
-Text Label 2200 4150 2    50   ~ 0
-GND
 $Comp
 L Connector_Generic:Conn_02x20_Odd_Even J1
@@
 Text Label 1000 2250 2    50   ~ 0
 3V3
-Text Label 1500 2250 0    50   ~ 0
-5V
 Text Label 1500 2450 0    50   ~ 0
 GND
@@
 INT
 Text Label 1000 2350 2    50   ~ 0
-3
+SDA
 Text Label 1000 2450 2    50   ~ 0
-5
+SCL
 Text Label 1000 2550 2    50   ~ 0
 7
 Text Label 1000 2750 2    50   ~ 0
-11
+ALRT
 Text Label 1000 2850 2    50   ~ 0
 13
@@
 Text Label 1500 4150 0    50   ~ 0
 40
-Text Label 1500 2350 0    50   ~ 0
+Text Label 1000 2650 2    50   ~ 0
+GND
+Text Label 1500 2850 0    50   ~ 0
+GND
+Text Label 1500 3150 0    50   ~ 0
+GND
+Text Label 1000 3450 2    50   ~ 0
+GND
+Text Label 1500 3650 0    50   ~ 0
+GND
+Text Label 1500 3850 0    50   ~ 0
+GND
+Text Label 1000 4150 2    50   ~ 0
+GND
+$Comp
+L Connector:Conn_01x10_Female J3
+U 1 1 5CA7DF40
+P 2650 2950
+F 0 "J3" H 2543 2325 50  0000 C CNN
+F 1 "ADS1115" H 2550 2200 50  0000 C CNN
+F 2 "Connector_PinHeader_2.54mm:PinHeader_1x10_P2.54mm_Vertical" H 2650 2950 50  0001 C CNN
+F 3 "~" H 2650 2950 50  0001 C CNN
+	1    2650 2950
+	1    0    0    1
+$EndComp
+Text Label 2450 3250 2    50   ~ 0
+GND
+Text Label 2450 3150 2    50   ~ 0
+SCL
+Text Label 2450 3050 2    50   ~ 0
+SDA
+Text Label 2450 2950 2    50   ~ 0
+GND
+Text Label 2450 2850 2    50   ~ 0
+ALRT
+Text Label 2450 2750 2    50   ~ 0
+A0
+Text Label 2450 2650 2    50   ~ 0
+A1
+Text Label 2450 2550 2    50   ~ 0
+A2
+Text Label 2450 2450 2    50   ~ 0
+A3
+$Comp
+L Connector:Conn_01x04_Male J2
+U 1 1 5CA8377C
+P 2400 3800
+F 0 "J2" H 2506 4078 50  0000 C CNN
+F 1 "Sensor input" H 2506 3987 50  0000 C CNN
+F 2 "Connector_PinHeader_2.54mm:PinHeader_1x04_P2.54mm_Vertical" H 2400 3800 50  0001 C CNN
+F 3 "~" H 2400 3800 50  0001 C CNN
+	1    2400 3800
+	1    0    0    -1
+$EndComp
+Text Label 2600 3700 0    50   ~ 0
+A0
+Text Label 2600 3800 0    50   ~ 0
+A1
+Text Label 2600 3900 0    50   ~ 0
+A2
+Text Label 2600 4000 0    50   ~ 0
+A3
+Text Label 2450 3350 2    50   ~ 0
+3V3
+$Comp
+L Connector:Conn_01x02_Male J7
+U 1 1 5CA84F35
+P 5500 1650
+F 0 "J7" H 5606 1828 50  0000 C CNN
+F 1 "Conn_01x02_Male" H 5606 1737 50  0000 C CNN
+F 2 "Connector_PinHeader_2.54mm:PinHeader_1x02_P2.54mm_Vertical" H 5500 1650 50  0001 C CNN
+F 3 "~" H 5500 1650 50  0001 C CNN
+	1    5500 1650
+	1    0    0    -1
+$EndComp
+Text Label 5700 1650 0    50   ~ 0
+CANH
+Text Label 5700 1750 0    50   ~ 0
+CANL
+Text Label 1500 2250 0    50   ~ 0
 5V
-Text Label 1000 2650 2    50   ~ 0
-GND
-Text Label 1500 2850 0    50   ~ 0
-GND
-Text Label 1500 3150 0    50   ~ 0
-GND
-Text Label 1000 3050 2    50   ~ 0
-3V3
-Text Label 1000 3450 2    50   ~ 0
-GND
-Text Label 1500 3650 0    50   ~ 0
-GND
-Text Label 1500 3850 0    50   ~ 0
-GND
-Text Label 1000 4150 2    50   ~ 0
-GND
 $EndSCHEMATC
